File: BM1368-1.kicad_sch (KiCad schematic)
At the start: 39 parts, among them U10 BM1370_mode1, U9 BM1370_mode1

Commit message: BOM specifications
Parts:
- C203, C204, C205, C27, C29, C31, C33, C34, C37, C40, C44, C46, C49, C60, C61, C65, C70, C71, C72, C73, C76, C78, C79, C80, C85, C93: value 1µ -> 1µ/25V; Brand (none) -> Samsung Electro-Mechanics; Distributor (none) -> D; Manufacturer (none) -> CL21B105KAFNNNE; OrderNr (none) -> 1276-1066-1-ND; Size (none) -> 0805
- C64, C68: value 10µ -> 10µ/25V; Brand (none) -> TDK Corporation; Size (none) -> 0805
- C74, C75: value 100n -> 100n/0.7mm; Brand (none) -> YAGEO; Distributor (none) -> D; Manufacturer (none) -> AC0805KRX7R9BB104; OrderNr (none) -> 311-3037-1-ND; Size (none) -> 0805
- C77: Brand (none) -> KEMET; Size (none) -> 1210
- R16, R19: Brand (none) -> Stackpole Electronics Inc; Distributor (none) -> D; Manufacturer (none) -> RNCP0805FTD1K00; OrderNr (none) -> RNCP0805FTD1K00CT-ND; Size (none) -> 0805
- R17, R20: Brand (none) -> Stackpole Electronics Inc; Distributor (none) -> D; Manufacturer (none) -> RMCF0805FT10K0; OrderNr (none) -> RMCF0805FT10K0CT-ND; Size (none) -> 0805
- R18, R49: Brand (none) -> TE Connectivity Passive Product; Distributor (none) -> D; Manufacturer (none) -> CRG0805F2K0; OrderNr (none) -> A126358CT-ND; Size (none) -> 0805
- U10, U9: Manufacturer (none) -> BITMAIN BM1370 ASIC
