File: BM1368-3.kicad_sch (KiCad schematic)
At the start: 39 parts, among them U13 BM1370_mode1, U14 BM1370_mode1

Commit message: BOM specifications
Parts:
- C148, C149, C150, C151, C152, C153, C154, C155, C156, C157, C158, C159, C161, C163, C164, C165, C166, C169, C171, C172, C173, C174, C175, C219, C220, C221: value 1µ -> 1µ/25V; Brand (none) -> Samsung Electro-Mechanics; Distributor (none) -> D; Manufacturer (none) -> CL21B105KAFNNNE; OrderNr (none) -> 1276-1066-1-ND; Size (none) -> 0805
- C160, C162: value 10µ -> 10µ/25V; Brand (none) -> TDK Corporation; Size (none) -> 0805
- C167, C168: value 100n -> 100n/0.7mm; Brand (none) -> YAGEO; Distributor (none) -> D; Manufacturer (none) -> AC0805KRX7R9BB104; OrderNr (none) -> 311-3037-1-ND; Size (none) -> 0805
- C170: Brand (none) -> KEMET; Size (none) -> 1210
- R42, R45: Brand (none) -> Stackpole Electronics Inc; Distributor (none) -> D; Manufacturer (none) -> RNCP0805FTD1K00; OrderNr (none) -> RNCP0805FTD1K00CT-ND; Size (none) -> 0805
- R43, R46: Brand (none) -> Stackpole Electronics Inc; Distributor (none) -> D; Manufacturer (none) -> RMCF0805FT10K0; OrderNr (none) -> RMCF0805FT10K0CT-ND; Size (none) -> 0805
- R44, R51: Brand (none) -> TE Connectivity Passive Product; Distributor (none) -> D; Manufacturer (none) -> CRG0805F2K0; OrderNr (none) -> A126358CT-ND; Size (none) -> 0805
- U13, U14: Manufacturer (none) -> BITMAIN BM1370 ASIC
