File: BM1368.kicad_sch (KiCad schematic)
At the start: 38 parts, among them U17 BM1370_mode1, U2 BM1370_mode1

Commit message: BOM specifications
Parts:
- C15, C17: value 10µ -> 10µ/25V; Brand (none) -> TDK Corporation; Size (none) -> 0805
- C195, C196, C197, C26, C28, C30, C32, C35, C36, C38, C41, C42, C43, C47, C50, C51, C52, C54, C56, C57, C58, C62, C63, C66, C67, C69: value 1µ -> 1µ/25V; Brand (none) -> Samsung Electro-Mechanics; Distributor (none) -> D; Manufacturer (none) -> CL21B105KAFNNNE; OrderNr (none) -> 1276-1066-1-ND; Size (none) -> 0805
- C53, C55: value 100n -> 100n/0.7mm; Brand (none) -> YAGEO; Distributor (none) -> D; Manufacturer (none) -> AC0805KRX7R9BB104; OrderNr (none) -> 311-3037-1-ND; Size (none) -> 0805
- C59: Brand (none) -> KEMET; Size (none) -> 1210
- R10, R15: Brand (none) -> Stackpole Electronics Inc; Distributor (none) -> D; Manufacturer (none) -> RMCF0805FT10K0; OrderNr (none) -> RMCF0805FT10K0CT-ND; Size (none) -> 0805
- R11: Brand (none) -> TE Connectivity Passive Product; Distributor (none) -> D; Manufacturer (none) -> CRG0805F2K0; OrderNr (none) -> A126358CT-ND; Size (none) -> 0805
- R14, R9: Brand (none) -> Stackpole Electronics Inc; Distributor (none) -> D; Manufacturer (none) -> RNCP0805FTD1K00; OrderNr (none) -> RNCP0805FTD1K00CT-ND; Size (none) -> 0805
- U17, U2: Manufacturer (none) -> BITMAIN BM1370 ASIC
