File: Nerd8.kicad_sch (KiCad schematic)
At the start: 3 parts, among them J1 Conn_01x04

Commit message: Added 4th Phase Buck
Started to add 4th Phase for the Buck, implementing BM1370 footprint etc
Other:
- sheet BM1368 renamed BM1370
Changed lines of the file:
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@@
 			(color 255 255 194 1.0000)
 		)
-		(property "Sheetname" "BM1368"
+		(property "Sheetname" "BM1370"
 			(at 82.55 90.7284 0)
 			(effects

Commit message: Changed LDO to 1V2 and original 1V2 to VDD
1V8 LDO replaced with 1V2 LDO
Crystal replaced
Other:
- sheet BM1370 ports: added VDD; removed +1V8
- sheet Power ports: added VDD; removed +1V8
Changed lines of the file:
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@@
 			)
 		)
-		(pin "+1V2" input
+		(pin "VDD" input
 			(at 82.55 97.79 180)
 			(effects
@@
 			)
 		)
-		(pin "+1V8" input
+		(pin "+1V2" input
 			(at 82.55 99.695 180)
 			(effects
@@
 			)
 		)
-		(pin "+1V2" output
+		(pin "VDD" output
 			(at 99.695 52.07 0)
 			(effects
@@
 			)
 		)
-		(pin "+1V8" output
+		(pin "+1V2" output
 			(at 99.695 53.975 0)
 			(effects

Commit message: Fuse from 12A to 15A
Parts:
- F1: value 12A -> 15A; Manufacturer 0451012.MRL -> 0451015.MRL; OrderNr F1228CT-ND -> F2593CT-ND
Changed lines of the file:
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@@
 			)
 		)
-		(property "Value" "12A"
+		(property "Value" "15A"
 			(at 50.165 49.3776 90)
 			(effects
@@
 			)
 		)
-		(property "Manufacturer" "0451012.MRL"
+		(property "Manufacturer" "0451015.MRL"
 			(at 50.165 52.07 0)
 			(effects
@@
 			)
 		)
-		(property "OrderNr" "F1228CT-ND"
+		(property "OrderNr" "F2593CT-ND"
 			(at 50.165 52.07 0)
 			(effects

Commit message: BOM specifications
Parts:
- D3: Brand (none) -> Littelfuse Inc.; Size (none) -> D_SMB
- F1: value 15A -> 20A; Brand (none) -> Littelfuse Inc.; Manufacturer 0451015.MRL -> 0451020.MRL; OrderNr F2593CT-ND -> F8251CT-ND
- J1: Brand (none) -> Amphenol Anytek; Size (none) -> 01x04
Changed lines of the file:
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@@
 			)
 		)
-		(property "Description" "Generic connector, single row, 01x04, script generated (kicad-library-utils/schlib/autogen/connector/)"
+		(property "Description" "CONN BARRIER STRIP 4CIRC 0.374\""
 			(at 27.94 46.99 0)
 			(effects
@@
 		)
 		(property "OrderNr" "YK5110403000G-ND"
+			(at 27.94 46.99 0)
+			(effects
+				(font
+					(size 1.27 1.27)
+				)
+				(hide yes)
+			)
+		)
+		(property "Brand" "Amphenol Anytek"
+			(at 27.94 46.99 0)
+			(effects
+				(font
+					(size 1.27 1.27)
+				)
+				(hide yes)
+			)
+		)
+		(property "Size" "01x04"
 			(at 27.94 46.99 0)
 			(effects
@@
 			)
 		)
-		(property "Description" ""
+		(property "Description" "TVS DIODE 12VWM 19.9VC DO214AA"
 			(at 55.245 58.42 0)
 			(effects
@@
 		)
 		(property "OrderNr" "SMBJ12ALFCT-ND"
+			(at 55.245 58.42 0)
+			(effects
+				(font
+					(size 1.27 1.27)
+				)
+				(hide yes)
+			)
+		)
+		(property "Brand" "Littelfuse Inc."
+			(at 55.245 58.42 0)
+			(effects
+				(font
+					(size 1.27 1.27)
+				)
+				(hide yes)
+			)
+		)
+		(property "Size" "D_SMB"
 			(at 55.245 58.42 0)
 			(effects
@@
 			)
 		)
-		(property "Value" "15A"
+		(property "Value" "20A"
 			(at 50.165 49.3776 90)
 			(effects
@@
 			)
 		)
-		(property "Description" ""
+		(property "Description" "FUSE BRD MNT 20A 65VAC 65VDC SMD"
 			(at 50.165 52.07 0)
 			(effects
@@
 			)
 		)
-		(property "Manufacturer" "0451015.MRL"
-			(at 50.165 52.07 0)
-			(effects
-				(font
-					(size 1.27 1.27)
-				)
-				(hide yes)
-			)
-		)
-		(property "OrderNr" "F2593CT-ND"
-			(at 50.165 52.07 0)
-			(effects
+		(property "Manufacturer" "0451020.MRL"
+			(at 50.165 52.07 0)
+			(effects
+				(font
+					(size 1.27 1.27)
+				)
+				(hide yes)
+			)
+		)
+		(property "OrderNr" "F8251CT-ND"
+			(at 50.165 52.07 0)
+			(effects
+				(font
+					(size 1.27 1.27)
+				)
+				(hide yes)
+			)
+		)
+		(property "Brand" "Littelfuse Inc."
+			(at 50.165 52.07 0)
+			(effects
+				(font
+					(size 1.27 1.27)
+				)
+				(hide yes)
+			)
+		)
+		(property "Size" ""
+			(at 50.165 52.07 0)
+			(effects
